Commit message: fixing joints

File: ros_ws/src/robot_description/urdf/arm_urdf.urdf (robot description, URDF)
Before this commit: robot arm_urdf, 5 links, 4 joints
Links:
- link base_link: geometry collision mesh filename=package://Arm Linkage model/meshes/base_link.STL; visual mesh filename=package://Arm Linkage model/meshes/base_link.STL
- link elbow: geometry collision mesh filename=package://Arm Linkage model/meshes/elbow.STL; visual mesh filename=package://Arm Linkage model/meshes/elbow.STL
- link shoulder: geometry collision mesh filename=package://Arm Linkage model/meshes/shoulder.STL; visual mesh filename=package://Arm Linkage model/meshes/shoulder.STL
- link wrist: geometry collision mesh filename=package://Arm Linkage model/meshes/wrist.STL; visual mesh filename=package://Arm Linkage model/meshes/wrist.STL
- link wrist_rotate: geometry collision mesh filename=package://Arm Linkage model/meshes/wrist_rotate.STL; visual mesh filename=package://Arm Linkage model/meshes/wrist_rotate.STL
Joints:
- joint elbow_joint: origin xyz=0.4572 0 0 rpy=0 0 -0.80481 -> xyz=0.35425 0 0.28903 rpy=0 0 0
- joint shoulder_joint: origin xyz=0.2958 -0.29557 0.467 rpy=1.5708 -0.68436 0 -> xyz=0.2958 -0.29557 0.467 rpy=0 0 0
- joint wrist_joint: origin xyz=0.508 0 0 rpy=0.12045 1.5708 0 -> xyz=0.50432 0 -0.061042 rpy=-3.1416 1.4178 -3.1416
- joint wrist_rotate_joint: origin xyz=-0.09 -0.063231 -0.0097485 rpy=-1.5437 -0.15297 1.5708 -> xyz=0.063978 -0.09 0 rpy=-1.5708 0 0

Commit message: renaming paths

File: ros_ws/src/robot_description/urdf/arm_urdf.urdf (robot description, URDF)
Before this commit: robot Arm Linkage model, 5 links, 4 joints
Links:
- link base_link: geometry collision mesh filename=package://robot_description/meshes/base_link.STL; visual mesh filename=package://robot_description/meshes/base_link.STL
- link elbow: geometry collision mesh filename=package://robot_description/meshes/elbow.STL; visual mesh filename=package://robot_description/meshes/elbow.STL
- link shoulder: geometry collision mesh filename=package://robot_description/meshes/shoulder.STL; visual mesh filename=package://robot_description/meshes/shoulder.STL
- link wrist: geometry collision mesh filename=package://robot_description/meshes/wrist.STL; visual mesh filename=package://robot_description/meshes/wrist.STL
- link wrist_rotate: geometry collision mesh filename=package://robot_description/meshes/wrist_rotate.STL; visual mesh filename=package://robot_description/meshes/wrist_rotate.STL

Commit message: fixing gripper joint

File: ros_ws/src/robot_description/urdf/arm_urdf.urdf (robot description, URDF)
Before this commit: robot robot_description, 6 links, 5 joints
Links:
- link gripper: mass 0.635591580584827 -> 0.635591580585097
Joints:
- removed joint gripper joint
- added joint gripper_joint: type revolute, parent arm_wrist, child gripper, origin xyz=0.014206 -0.078774 -0.024953 rpy=0 0 0, axis 1 0 0, limit lower=-3.14 upper=3.14 effort=10 velocity=10

Commit message: 2nd fix for gripper

File: ros_ws/src/robot_description/urdf/arm_urdf.urdf (robot description, URDF)
Before this commit: robot robot_description, 6 links, 5 joints
Links:
- link gripper: mass 0.635591580585097 -> 0.635591580585016
