Commit message: adding depth camera and imu to sim

File: ros_ws/src/robot_description/urdf/gazebo.xacro (robot description, xacro)
@@ -1,4 +1,4 @@
 <?xml version="1.0" ?>
-<robot name="zinger" xmlns:xacro="http://www.ros.org/wiki/xacro" >
+<robot name="robot_description" xmlns:xacro="http://www.ros.org/wiki/xacro" >
     <!--
         GAZEBO MACROS
@@ -20,4 +20,119 @@
         </gazebo>
     </xacro:macro>
+    <gazebo reference="intel_realsense">
+        <sensor name="intel_realsense_depth" type="depth_camera">
+            <always_on>1</always_on>
+            <update_rate>20</update_rate>
+            <pose>0 0 0 0 0 -1.57</pose>
+            <topic>intel_realsense</topic>
+            <camera name="realsense_depth_camera">
+                <horizontal_fov>1.02974</horizontal_fov>
+                <clip>
+                    <near>0.02</near>
+                    <far>20</far>
+                </clip>
+                <noise>
+                    <type>gaussian</type>
+                    <mean>0.0</mean>
+                    <stddev>0.007</stddev>
+                </noise>
+            </camera>
+            <plugin
+                filename="libignition-gazebo-sensors-system.so"
+                name="ignition::gazebo::systems::Sensors">
+                <render_engine>ogre2</render_engine>
+            </plugin>
+        </sensor>
+        <!-- <sensor name="intel_realsense_rgb" type="rgbd_camera">
+            <always_on>true</always_on>
+            <visualize>false</visualize>
+            <update_rate>5</update_rate>
+            <topic>intel_realsense</topic>
+            <enable_metrics>true</enable_metrics>
+            <pose>0 0 0 0 0 0</pose>
+            <camera name="realsense_rgb_camera">
+            <horizontal_fov>1.02974</horizontal_fov>
+            <image>
+                <width>1920</width>
+                <height>1080</height>
+                <format>RGB_INT8</format>
+            </image>
+            <clip>
+                <near>0.02</near>
+                <far>20</far>
+            </clip>
+            <depth_camera>
+                <clip>
+                    <near>0.05</near>
+                    <far>20.0</far>
+                </clip>
+            </depth_camera>
+            <noise>
+                <type>gaussian</type>
+                <mean>0.0</mean>
+                <stddev>0.007</stddev>
+            </noise>
+            </camera>
+            <plugin
+                filename="libignition-gazebo-sensors-system.so"
+                name="ignition::gazebo::systems::Sensors">
+                <render_engine>ogre2</render_engine>
+            </plugin>
+        </sensor> -->
+        <sensor name="imu_sensor" type="imu">
+            <ignition_frame_id>intel_realsense</ignition_frame_id>
+            <always_on>true</always_on>
+            <update_rate>25</update_rate>
+            <imu>
+                <angular_velocity>
+                <x>
+                    <noise type="gaussian">
+                    <mean>0.0</mean>
+                    <stddev>0.0</stddev>
+                    </noise>
+                </x>
+                <y>
+                    <noise type="gaussian">
+                    <mean>0.0</mean>
+                    <stddev>0.0</stddev>
+                    </noise>
+                </y>
+                <z>
+                    <noise type="gaussian">
+                    <mean>0.0</mean>
+                    <stddev>0.0</stddev>
+                    </noise>
+                </z>
+                </angular_velocity>
+                <linear_acceleration>
+                <x>
+                    <noise type="gaussian">
+                    <mean>0.0</mean>
+                    <stddev>0.0</stddev>
+                    </noise>
+                </x>
+                <y>
+                    <noise type="gaussian">
+                    <mean>0.0</mean>
+                    <stddev>0.0</stddev>
+                    </noise>
+                </y>
+                <z>
+                    <noise type="gaussian">
+                    <mean>0.0</mean>
+                    <stddev>0.0</stddev>
+                    </noise>
+                </z>
+                </linear_acceleration>
+            </imu>
+            <plugin
+                filename="libignition-gazebo-imu-system.so"
+                name="ignition::gazebo::systems::Imu">
+                <alwaysOn>true</alwaysOn>
+                <updateRate>25</updateRate>
+                <topic>imu</topic>
+            </plugin>
+        </sensor>
+    </gazebo>
     <!--
         GAZEBO

File: ros_ws/src/robot_description/urdf/robot_description.urdf (robot description, URDF)
Before this commit: robot robot_description, 9 links, 8 joints
Links:
- added link intel_realsense, mass ${mass}; collision box size=${length_x} ${length_y} ${length_z}; visual box size=${length_x} ${length_y} ${length_z}
Joints:
- added joint intel_realsense_joint: type fixed, parent chassis, child intel_realsense, origin xyz=0.95 -0.5 1.5 rpy=0 0 0
