Commit message: adding how the depth cam works on turtlebot but commenting since it wasn't working with ignition

File: ros_ws/src/robot_description/urdf/depth_camera.xacro (robot description, xacro)
@@ -32,3 +32,57 @@
         <origin rpy="0 0 0" xyz="0.95 -0.5 1.5" />
     </joint>
+    <!-- ************** -->
+    <!-- <link name="camera_link"/>
+    <link name="camera_rgb_optical_frame">
+      <inertial>
+        <origin xyz="0.069 -0.047 0.107" rpy="0 0 0"/>
+        <mass value="0.035"/>
+        <inertia ixx="0.001" ixy="0.000" ixz="0.000" iyy="0.001" iyz="0.000" izz="0.001"/>
+      </inertial>
+    </link>
+    <joint name="camera_joint" type="fixed">
+      <parent link="chassis"/>
+      <child link="camera_link"/>
+      <origin xyz="0.95 -0.5 1.5" rpy="0 0 0"/>
+    </joint>
+    <joint name="camera_rgb_joint" type="fixed">
+      <parent link="camera_link"/>
+      <child link="camera_rgb_frame"/>
+      <origin xyz="0.005 0.018 0.013" rpy="0 0 0"/>
+    </joint>
+    <joint name="camera_rgb_optical_joint" type="fixed">
+      <parent link="camera_rgb_frame"/>
+      <child link="camera_rgb_optical_frame"/>
+      <origin xyz="0 0 0" rpy="-1.57079632679 0 -1.57079632679"/>
+    </joint>
+    <link name="camera_rgb_frame"/>
+    <gazebo reference="camera_rgb_optical_frame">
+        <sensor name="camera" type="depth">
+            <always_on>true</always_on>
+            <visualize>true</visualize>
+            <update_rate>30</update_rate>
+            <camera name="intel_realsense_r200">
+            <horizontal_fov>1.51</horizontal_fov>
+            <vertical_fov>1.01</vertical_fov>
+            <image>
+                <width>640</width>
+                <height>480</height>
+                <format>R8G8B8</format>
+            </image>
+            <clip>
+                <near>0.2</near>
+                <far>8</far>
+            </clip>
+            <noise>
+                <type>gaussian</type>
+                <mean>0.0</mean>
+                <stddev>0.007</stddev>
+            </noise>
+            </camera>
+            <plugin name="camera_driver" filename="libgazebo_ros_camera.so">
+            <ros>
+            </ros>
+            </plugin>
+        </sensor>
+    </gazebo> -->
 </robot>
