Commit message: adding indents

File: ros_ws/src/robot_description/urdf/wheels.xacro (robot description, xacro)
@@ -27,9 +27,9 @@
     </link>
     <joint name="rear_right_swerve_joint" type="revolute">
-    <origin xyz="0.68344 -0.49838 0.7682" rpy="0 0 -1.5703" />
-    <parent link="chassis" />
-    <child link="rear_right_swerve" />
-    <axis xyz="0 0 1" />
-    <limit lower="-3.14" upper="3.14" effort="10" velocity="10" />
+        <origin xyz="0.68344 -0.49838 0.7682" rpy="0 0 -1.5703" />
+        <parent link="chassis" />
+        <child link="rear_right_swerve" />
+        <axis xyz="0 0 1" />
+        <limit lower="-3.14" upper="3.14" effort="10" velocity="10" />
     </joint>
     <link name="rear_right_wheel">
@@ -57,9 +57,9 @@
     </link>
     <joint name="rear_right_wheel_joint" type="continuous">
-    <origin xyz="0 0.00025221 -0.123" rpy="0 0 0" />
-    <parent link="rear_right_swerve" />
-    <child link="rear_right_wheel" />
-    <axis xyz="0 1 0" />
-    <limit lower="0" upper="0" effort="10" velocity="10" />
+        <origin xyz="0 0.00025221 -0.123" rpy="0 0 0" />
+        <parent link="rear_right_swerve" />
+        <child link="rear_right_wheel" />
+        <axis xyz="0 1 0" />
+        <limit lower="0" upper="0" effort="10" velocity="10" />
     </joint>
     <link name="rear_left_swerve">
@@ -87,9 +87,9 @@
     </link>
     <joint name="rear_left_swerve_joint" type="revolute">
-    <origin xyz="1.2863 -0.49838 0.7682" rpy="0 0 -1.5703" />
-    <parent link="chassis" />
-    <child link="rear_left_swerve" />
-    <axis xyz="0 0 1" />
-    <limit lower="-3.14" upper="3.14" effort="10" velocity="10" />
+        <origin xyz="1.2863 -0.49838 0.7682" rpy="0 0 -1.5703" />
+        <parent link="chassis" />
+        <child link="rear_left_swerve" />
+        <axis xyz="0 0 1" />
+        <limit lower="-3.14" upper="3.14" effort="10" velocity="10" />
     </joint>
     <link name="rear_left_wheel">
@@ -117,9 +117,9 @@
     </link>
     <joint name="rear_left_wheel_joint" type="continuous">
-    <origin xyz="0 -0.00025221 -0.123" rpy="0 0 0" />
-    <parent link="rear_left_swerve" />
-    <child link="rear_left_wheel" />
-    <axis xyz="0 1 0" />
-    <limit effort="10" velocity="10" />
+        <origin xyz="0 -0.00025221 -0.123" rpy="0 0 0" />
+        <parent link="rear_left_swerve" />
+        <child link="rear_left_wheel" />
+        <axis xyz="0 1 0" />
+        <limit effort="10" velocity="10" />
     </joint>
     <link name="front_left_swerve">
@@ -147,9 +147,9 @@
     </link>
     <joint name="front_left_swerve_joint" type="revolute">
-    <origin xyz="1.2863 -1.4072 0.77214" rpy="0 0 -1.5703" />
-    <parent link="chassis" />
-    <child link="front_left_swerve" />
-    <axis xyz="0 0 1" />
-    <limit lower="-3.14" upper="3.14" effort="10" velocity="10" />
+        <origin xyz="1.2863 -1.4072 0.77214" rpy="0 0 -1.5703" />
+        <parent link="chassis" />
+        <child link="front_left_swerve" />
+        <axis xyz="0 0 1" />
+        <limit lower="-3.14" upper="3.14" effort="10" velocity="10" />
     </joint>
     <link name="front_left_wheel">
@@ -177,9 +177,9 @@
     </link>
     <joint name="front_left_wheel_joint" type="continuous">
-    <origin xyz="0 -0.00025221 -0.12694" rpy="0 0 0" />
-    <parent link="front_left_swerve" />
-    <child link="front_left_wheel" />
-    <axis xyz="0 1 0" />
-    <limit effort="10" velocity="10" />
+        <origin xyz="0 -0.00025221 -0.12694" rpy="0 0 0" />
+        <parent link="front_left_swerve" />
+        <child link="front_left_wheel" />
+        <axis xyz="0 1 0" />
+        <limit effort="10" velocity="10" />
     </joint>
     <link name="front_right_swerve">
@@ -207,9 +207,9 @@
     </link>
     <joint name="front_right_swerve_joint" type="revolute">
-    <origin xyz="0.68344 -1.4072 0.76536" rpy="0 0 -1.5703" />
-    <parent link="chassis" />
-    <child link="front_right_swerve" />
-    <axis xyz="0 0 1" />
-    <limit lower="-3.14" upper="3.14" effort="10" velocity="10" />
+        <origin xyz="0.68344 -1.4072 0.76536" rpy="0 0 -1.5703" />
+        <parent link="chassis" />
+        <child link="front_right_swerve" />
+        <axis xyz="0 0 1" />
+        <limit lower="-3.14" upper="3.14" effort="10" velocity="10" />
     </joint>
     <link name="front_right_wheel">
@@ -237,9 +237,9 @@
     </link>
     <joint name="front_right_wheel_joint" type="continuous">
-    <origin xyz="0 0.00025221 -0.12016" rpy="0 0 0" />
-    <parent link="front_right_swerve" />
-    <child link="front_right_wheel" />
-    <axis xyz="0 1 0" />
-    <limit effort="10" velocity="10" />
+        <origin xyz="0 0.00025221 -0.12016" rpy="0 0 0" />
+        <parent link="front_right_swerve" />
+        <child link="front_right_wheel" />
+        <axis xyz="0 1 0" />
+        <limit effort="10" velocity="10" />
     </joint>
 </robot>
