Commit message: initial commit for gazebo sim

File: ros_ws/src/robot_description/urdf/robot_description.urdf (robot description, URDF)
Before this commit: robot robot_description, 9 links, 8 joints
Links:
- link chassis: mass 9.00191258390929 -> 3.00191258390929
- link front_left_wheel: mass 0.656482054320522 -> 3.656482054320522
- link front_right_wheel: mass 0.656482054320521 -> 3.656482054320521

Commit message: adding base link

File: ros_ws/src/robot_description/urdf/robot_description.urdf (robot description, URDF)
Before this commit: robot robot_description, 9 links, 8 joints
Links:
- added link base_link
Joints:
- added joint joint_chassis_to_base: type fixed, parent chassis, child base_link, origin xyz=0.98467 -1.02594 0.94417 rpy=0 0 -1.57079633

Commit message: Simplifying the robot description into their own named xacro files

File: ros_ws/src/robot_description/urdf/robot_description.urdf (robot description, URDF)
Before this commit: robot robot_description, 12 links, 11 joints
Links:
- removed link front_left_swerve
- removed link front_left_wheel
- removed link front_right_swerve
- removed link front_right_wheel
- removed link imu_sensor_link
- removed link intel_realsense
- removed link rear_left_swerve
- removed link rear_left_wheel
- removed link rear_right_swerve
- removed link rear_right_wheel
Joints:
- removed joint base_link_to_imu
- removed joint front_left_swerve_joint
- removed joint front_left_wheel_joint
- removed joint front_right_swerve_joint
- removed joint front_right_wheel_joint
- removed joint intel_realsense_joint
- removed joint rear_left_swerve_joint
- removed joint rear_left_wheel_joint
- removed joint rear_right_swerve_joint
- removed joint rear_right_wheel_joint

Commit message: adding a base_footprint frame to the robot

File: ros_ws/src/robot_description/urdf/robot_description.urdf (robot description, URDF)
Before this commit: robot robot_description, 2 links, 1 joints
Links:
- added link base_footprint
Joints:
- added joint base_footprint_joint: type fixed, parent base_link, child base_footprint, origin xyz=0 0 -0.40 rpy=0 0 0

Commit message: angle updates

File: ros_ws/src/robot_description/urdf/robot_description.urdf (robot description, URDF)
Before this commit: robot robot_description, 9 links, 8 joints
Links:
- removed link chassis
- removed link front_left_swerve
- removed link front_left_wheel
- removed link front_right_swerve
- removed link front_right_wheel
- removed link rear_left_swerve
- removed link rear_left_wheel
- removed link rear_right_swerve
- removed link rear_right_wheel
- added link arm_base, mass 3.22741129215856; collision mesh filename=package://robot_description/meshes/arm_base.STL; visual mesh filename=package://robot_description/meshes/arm_base.STL
- added link arm_base_footprint, mass 119.491304287739; collision mesh filename=package://robot_description/meshes/arm_base_footprint.STL; visual mesh filename=package://robot_description/meshes/arm_base_footprint.STL
- added link arm_elbow, mass 1.84402735327987; collision mesh filename=package://robot_description/meshes/arm_elbow.STL; visual mesh filename=package://robot_description/meshes/arm_elbow.STL
- added link arm_shoulder, mass 0.974957548893572; collision mesh filename=package://robot_description/meshes/arm_shoulder.STL; visual mesh filename=package://robot_description/meshes/arm_shoulder.STL
- added link arm_wrist, mass 0.266662965128272; collision mesh filename=package://robot_description/meshes/arm_wrist.STL; visual mesh filename=package://robot_description/meshes/arm_wrist.STL
- added link gripper, mass 0.635591580584878; collision mesh filename=package://robot_description/meshes/gripper.STL; visual mesh filename=package://robot_description/meshes/gripper.STL
Joints:
- removed joint front_left_swerve_joint
- removed joint front_left_wheel_joint
- removed joint front_right_swerve_joint
- removed joint front_right_wheel_joint
- removed joint rear_left_swerve_joint
- removed joint rear_left_wheel_joint
- removed joint rear_right_swerve_joint
- removed joint rear_right_wheel_joint
- added joint arm_base_joint: type revolute, parent arm_base_footprint, child arm_base, origin xyz=0.025047 -0.11824 0.13851 rpy=0 0 0.049606, axis 0 0 1, limit lower=-3.14 upper=3.14 effort=10 velocity=10
- added joint arm_elbow_joint: type revolute, parent arm_shoulder, child arm_elbow, origin xyz=-0.22191 -0.00635 0.25014 rpy=-1.5708 -1.3963 3.1416, axis 0 1 0, limit lower=-1.57 upper=1.57 effort=10 velocity=10
- added joint arm_shoulder_joint: type revolute, parent arm_base, child arm_shoulder, origin xyz=0.0635 -0.19367 0.3277 rpy=3.1416 0.3735 1.5212, axis 0 1 0, limit lower=-1.57 upper=1.57 effort=10 velocity=10
- added joint arm_wrist_joint: type revolute, parent arm_elbow, child arm_wrist, origin xyz=0.2358 -0.019078 0.028575 rpy=0 0 2.2066, axis 0 1 0, limit lower=-1.57 upper=1.57 effort=10 velocity=10
- added joint gripper joint: type revolute, parent arm_wrist, child gripper, origin xyz=0.0051746 -0.075951 0.035385 rpy=-3.1368 0 1.5708, axis 1 0 0, limit lower=-1.57 upper=1.57 effort=10 velocity=10

Commit message: fixing angle update

File: ros_ws/src/robot_description/urdf/robot_description.urdf (robot description, URDF)
Before this commit: robot robot_description, 6 links, 5 joints
Links:
- link arm_shoulder: mass 0.974957548893572 -> 0.974957548893571
Joints:
- joint arm_base_joint: limit lower=-3.14 upper=3.14 effort=10 velocity=10 -> lower=-1.57 upper=1.57 effort=10 velocity=10; origin xyz=0.025047 -0.11824 0.13851 rpy=0 0 0.049606 -> xyz=0.025047 -0.11824 0.13851 rpy=0 0 -1.5708
- joint arm_elbow_joint: origin xyz=-0.22191 -0.00635 0.25014 rpy=-1.5708 -1.3963 3.1416 -> xyz=0.42568 0.003175 0.16682 rpy=0 0 0
- joint arm_shoulder_joint: origin xyz=0.0635 -0.19367 0.3277 rpy=3.1416 0.3735 1.5212 -> xyz=-0.06985 -0.079375 0.22575 rpy=0 0 0
- joint arm_wrist_joint: origin xyz=0.2358 -0.019078 0.028575 rpy=0 0 2.2066 -> xyz=0.26467 0 -0.4336 rpy=0 0 0
- joint gripper joint: origin xyz=0.0051746 -0.075951 0.035385 rpy=-3.1368 0 1.5708 -> xyz=0.004356 0.074295 -0.0010894 rpy=0 0 0
