Commit message: refactoring urdf files

File: ros_ws/src/robot_description/urdf/arm.urdf (robot description, URDF)
Before this commit: robot arm, 6 links, 5 joints
Links:
- link arm_base: mass 3.22741129192052 -> 3.22741129215856
- link arm_base_footprint: mass 135.989046906803 -> 119.491304287739
- link gripper: mass 0.635591580585016 -> 0.635591580584878
Joints:
- joint arm_base_joint: limit lower=-3.14 upper=3.14 effort=10 velocity=10 -> lower=-1.57 upper=1.57 effort=10 velocity=10; origin xyz=0.11824 0.025047 0.13851 rpy=0 0 0 -> xyz=0.025047 -0.11824 0.13851 rpy=0 0 -1.5708
- joint arm_elbow_joint: axis 0 1 0 -> 0 -1 0; origin xyz=0.25455 0.13544 0.3837 rpy=0 0 0 -> xyz=0.42568 0.003175 0.16682 rpy=0 0 0
- joint arm_shoulder_joint: axis 0 1 0 -> 0 -1 0; origin xyz=-0.072332 -0.057326 0.22575 rpy=0 0 0 -> xyz=-0.06985 -0.079375 0.22575 rpy=0 0 0
- joint arm_wrist_joint: origin xyz=0.49451 -0.030405 -0.11266 rpy=0 0 0 -> xyz=0.26467 0 -0.4336 rpy=0 0 0
- joint gripper_joint: limit lower=-3.14 upper=3.14 effort=10 velocity=10 -> lower=-1.57 upper=1.57 effort=10 velocity=10; origin xyz=0.014206 -0.078774 -0.024953 rpy=0 0 0 -> xyz=0.004356 0.074295 -0.0010894 rpy=0 0 0

Commit message: changes based on hardware testing

File: ros_ws/src/robot_description/urdf/arm.urdf (robot description, URDF)
Before this commit: robot arm, 6 links, 5 joints
Joints:
- joint arm_shoulder_joint: limit lower=-1.57 upper=1.57 effort=10 velocity=10 -> lower=-1.57 upper=0.667 effort=10 velocity=10

Commit message: more changes from hardware

File: ros_ws/src/robot_description/urdf/arm.urdf (robot description, URDF)
Before this commit: robot arm, 6 links, 5 joints
Joints:
- joint arm_elbow_joint: limit lower=-1.57 upper=1.57 effort=10 velocity=10 -> lower=0 upper=0.8 effort=10 velocity=10

Commit message: Remove RAD encoder feedback from arm and tweaking joint limits

File: ros_ws/src/robot_description/urdf/arm.urdf (robot description, URDF)
Before this commit: robot arm, 6 links, 5 joints
Joints:
- joint arm_elbow_joint: axis 0 -1 0 -> 0 1 0

Commit message: updating wrist joints with inital positions

File: ros_ws/src/robot_description/urdf/arm.urdf (robot description, URDF)
Before this commit: robot arm, 6 links, 5 joints
Links:
- link arm_base: mass 3.22741129192052 -> 3.22741129215856
- link arm_base_footprint: mass 135.989046906803 -> 119.491304287739
- link arm_shoulder: mass 0.974957548893571 -> 0.974957548893572
- link arm_wrist: mass 0.266662965128272 -> 0.266662965128273
- link gripper: mass 0.635591580585016 -> 0.635591580584949
Joints:
- removed joint gripper_joint
- added joint gripper joint: type revolute, parent arm_wrist, child gripper, origin xyz=0.0038697 0.074295 0.0022774 rpy=0 -0.39004 0, axis 1 0 0, limit lower=-1.57 upper=1.57 effort=10 velocity=10
- joint arm_base_joint: limit lower=-3.14 upper=3.14 effort=10 velocity=10 -> lower=-1.57 upper=1.57 effort=10 velocity=10; origin xyz=0.11824 0.025047 0.13851 rpy=0 0 0 -> xyz=0.025047 -0.11824 0.13851 rpy=0 0 -1.5708
- joint arm_elbow_joint: limit lower=-1.57 upper=1.57 effort=10 velocity=10 -> lower=0 upper=0.8 effort=10 velocity=10; origin xyz=0.25455 0.13544 0.3837 rpy=0 0 0 -> xyz=0.42568 0.003175 0.16682 rpy=0 0 0
- joint arm_shoulder_joint: axis 0 1 0 -> 0 -1 0; limit lower=-1.57 upper=1.57 effort=10 velocity=10 -> lower=-1.57 upper=0.667 effort=10 velocity=10; origin xyz=-0.072332 -0.057326 0.22575 rpy=0 0 0 -> xyz=-0.06985 -0.079375 0.22575 rpy=0 0 0
- joint arm_wrist_joint: limit lower=-1.57 upper=1.57 effort=10 velocity=10 -> lower=0 upper=1.57 effort=10 velocity=10; origin xyz=0.49451 -0.030405 -0.11266 rpy=0 0 0 -> xyz=0.26467 0 -0.4336 rpy=0 0 0

Commit message: changes after testing

File: ros_ws/src/robot_description/urdf/arm.urdf (robot description, URDF)
Before this commit: robot arm, 6 links, 5 joints
Joints:
- removed joint gripper joint
- added joint gripper_joint: type revolute, parent arm_wrist, child gripper, origin xyz=0.0038697 0.074295 0.0022774 rpy=0 -0.39004 0, axis -1 0 0, limit lower=0 upper=3.14 effort=10 velocity=10

Commit message: changing wrist direction in urdf

File: ros_ws/src/robot_description/urdf/arm.urdf (robot description, URDF)
Before this commit: robot arm, 6 links, 5 joints
Joints:
- joint arm_wrist_joint: axis 0 1 0 -> 0 -1 0; limit lower=0 upper=1.57 effort=10 velocity=10 -> lower=-1.57 upper=0 effort=10 velocity=10
